File: SourceControlTest.kicad_sch (KiCad schematic)
At the start: 0 parts

Commit message: Added Basic LC1 Circuit
Parts:
- added C1: 10uF, symbol Device:C
- added R1: 20k, symbol Device:R_US
- added R2: 10k, symbol Device:R_US
- added Vs: 10v, symbol Device:Battery_Cell
Connections:
- new net: C1.1, R1.1, Vs.1 (+)
- new net: R1.2, R2.1
- new net GND: C1.2, R2.2, Vs.2 (-)

Commit message: Learned Hiercheries
Connections:
- net SecondDivider/Division_In: now reaches R1.2, R2.1
Other:
- added sheet SecondDivider (seconddivider.kicad_sch)
Changed lines of the file:
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@@
 	(paper "A4")
+	(junction
+		(at 152.4 90.17)
+		(diameter 0)
+		(color 0 0 0 0)
+	)
 	(junction
 		(at 128.27 101.6)
@@
 		(color 0 0 0 0)
 	)
+	(junction
+		(at 152.4 100.33)
+		(diameter 0)
+		(color 0 0 0 0)
+	)
 	(wire
 		(pts
@@
 	(wire
 		(pts
-			(xy 152.4 88.9) (xy 152.4 91.44)
+			(xy 152.4 100.33) (xy 158.75 100.33)
+		)
+		(stroke
+			(width 0)
+			(type default)
+		)
+	)
+	(wire
+		(pts
+			(xy 152.4 88.9) (xy 152.4 90.17)
 		)
 		(stroke
@@
 	(wire
 		(pts
+			(xy 152.4 100.33) (xy 152.4 99.06)
+		)
+		(stroke
+			(width 0)
+			(type default)
+		)
+	)
+	(wire
+		(pts
 			(xy 114.3 88.9) (xy 128.27 88.9)
 		)
@@
 	(wire
 		(pts
+			(xy 152.4 90.17) (xy 152.4 91.44)
+		)
+		(stroke
+			(width 0)
+			(type default)
+		)
+	)
+	(wire
+		(pts
 			(xy 128.27 88.9) (xy 134.62 88.9)
 		)
@@
 	(wire
 		(pts
+			(xy 152.4 90.17) (xy 158.75 90.17)
+		)
+		(stroke
+			(width 0)
+			(type default)
+		)
+	)
+	(wire
+		(pts
 			(xy 114.3 99.06) (xy 114.3 101.6)
 		)
@@
 	(wire
 		(pts
-			(xy 152.4 101.6) (xy 152.4 99.06)
+			(xy 152.4 101.6) (xy 152.4 100.33)
 		)
 		(stroke
@@
 				)
 			)
+		)
+	)
+	(sheet
+		(at 158.75 88.9)
+		(size 20.32 12.7)
+		(exclude_from_sim no)
+		(in_bom yes)
+		(on_board yes)
+		(dnp no)
+		(stroke
+			(width 0.1524)
+			(type solid)
+		)
+		(fill
+			(color 0 0 0 0)
+		)
+		(property "Sheetname" "SecondDivider"
+			(at 158.496 86.106 0)
+			(show_name no)
+			(do_not_autoplace no)
+			(effects
+				(font
+					(size 1.27 1.27)
+				)
+				(justify left bottom)
+			)
+		)
+		(property "Sheetfile" "seconddivider.kicad_sch"
+			(at 158.496 87.122 0)
+			(show_name no)
+			(do_not_autoplace no)
+			(effects
+				(font
+					(size 1.27 1.27)
+				)
+				(justify left top)
+			)
+		)
+		(pin "Division_In" input
+			(at 158.75 90.17 180)
+			(effects
+				(font
+					(size 1.27 1.27)
+				)
+				(justify left)
+			)
+		)
+		(pin "GND" input
+			(at 158.75 100.33 180)
+			(effects
+				(font
+					(size 1.27 1.27)
+				)
+				(justify left)
+			)
+		)
+		(pin "Voltage_Output" output
+			(at 179.07 95.25 0)
+			(effects
+				(font
+					(size 1.27 1.27)
+				)
+				(justify right)
+			)
+		)
+		(instances
+			(project "SourceControlTest"
+				(path "/5d981c2c-ab3d-4850-ba6d-abf03e2cd683"
+					(page "2")
+				)
+			)

Commit message: messed with pcb
Parts:
- C1: footprint (none) -> Capacitor_SMD:CP_Elec_3x5.3
- R1, R2: footprint (none) -> Resistor_THT:R_Axial_DIN0309_L9.0mm_D3.2mm_P2.54mm_Vertical
- Vs1: renamed from Vs; footprint (none) -> Connector_Phoenix_MC_HighVoltage:PhoenixContact_MCV_1,5_2-G-5.08_1x02_P5.08mm_Vertical
Changed lines of the file:
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@@
 			)
 		)
-		(property "Footprint" ""
+		(property "Footprint" "Capacitor_SMD:CP_Elec_3x5.3"
 			(at 129.2352 99.06 0)
 			(hide yes)
@@
 			)
 		)
-		(property "Footprint" ""
+		(property "Footprint" "Resistor_THT:R_Axial_DIN0309_L9.0mm_D3.2mm_P2.54mm_Vertical"
 			(at 138.684 87.884 90)
 			(hide yes)
@@
 			)
 		)
-		(property "Footprint" ""
+		(property "Footprint" "Resistor_THT:R_Axial_DIN0309_L9.0mm_D3.2mm_P2.54mm_Vertical"
 			(at 153.416 95.504 90)
 			(hide yes)
@@
 		(in_pos_files yes)
 		(dnp no)
-		(property "Reference" "Vs"
+		(property "Reference" "Vs1"
 			(at 111.252 94.234 0)
 			(show_name no)
@@
 			)
 		)
-		(property "Footprint" ""
+		(property "Footprint" "Connector_Phoenix_MC_HighVoltage:PhoenixContact_MCV_1,5_2-G-5.08_1x02_P5.08mm_Vertical"
 			(at 114.3 94.996 90)
 			(hide yes)
@@
 			(project "SourceControlTest"
 				(path "/5d981c2c-ab3d-4850-ba6d-abf03e2cd683"
-					(reference "Vs")
-					(unit 1)
-				)
+					(reference "Vs1")
+					(unit 1)
+				)
