File: SourceControlTest.kicad_pcb (KiCad board)
At the start: 2 copper layers, 6 parts

Commit message: extra
Parts:
- moved R4 54.5 mm to (112.1, 74.5)
- moved R1 44.7 mm to (96.5, 74.5)
- moved R3 40.9 mm to (120.0, 80.0), turned to -90 degrees
Routing:
- net GND: track 0.00 -> 3.00 mm
Changed lines of the file:
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@@
 	(footprint "Resistor_THT:R_Axial_DIN0309_L9.0mm_D3.2mm_P2.54mm_Vertical"
 		(layer "F.Cu")
-		(at 140.63 81.5)
+		(at 96.46 74.5)
 		(descr "Resistor, Axial_DIN0309 series, Axial, Vertical, pin pitch=2.54mm, 0.5W = 1/2W, length*diameter=9*3.2mm^2, http://cdn-reichelt.de/documents/datenblatt/B400/1_4W%23YAG.pdf")
 		(tags "Resistor Axial_DIN0309 series Axial Vertical pin pitch 2.54mm 0.5W = 1/2W length 9mm diameter 3.2mm")
@@
 	(footprint "Resistor_THT:R_Axial_DIN0309_L9.0mm_D3.2mm_P2.54mm_Vertical"
 		(layer "F.Cu")
-		(at 158.63 103)
+		(at 112.13 74.5)
 		(descr "Resistor, Axial_DIN0309 series, Axial, Vertical, pin pitch=2.54mm, 0.5W = 1/2W, length*diameter=9*3.2mm^2, http://cdn-reichelt.de/documents/datenblatt/B400/1_4W%23YAG.pdf")
 		(tags "Resistor Axial_DIN0309 series Axial Vertical pin pitch 2.54mm 0.5W = 1/2W length 9mm diameter 3.2mm")
@@
 	(footprint "Resistor_THT:R_Axial_DIN0309_L9.0mm_D3.2mm_P2.54mm_Vertical"
 		(layer "F.Cu")
-		(at 159.63 90)
+		(at 120 79.96 -90)
 		(descr "Resistor, Axial_DIN0309 series, Axial, Vertical, pin pitch=2.54mm, 0.5W = 1/2W, length*diameter=9*3.2mm^2, http://cdn-reichelt.de/documents/datenblatt/B400/1_4W%23YAG.pdf")
 		(tags "Resistor Axial_DIN0309 series Axial Vertical pin pitch 2.54mm 0.5W = 1/2W length 9mm diameter 3.2mm")
 		(property "Reference" "R3"
-			(at 1.27 -2.72 0)
+			(at 1.27 -2.72 90)
 			(layer "F.SilkS")
 			(effects
@@
 		)
 		(property "Value" "R_US"
-			(at 1.27 2.72 0)
+			(at 1.27 2.72 90)
 			(layer "F.Fab")
 			(effects
@@
 		)
 		(property "Datasheet" ""
-			(at 0 0 0)
+			(at 0 0 90)
 			(layer "F.Fab")
 			(hide yes)
@@
 		)
 		(property "Description" "Resistor, US symbol"
-			(at 0 0 0)
+			(at 0 0 90)
 			(layer "F.Fab")
 			(hide yes)
@@
 		)
 		(property "KiLib_Generator" "resistor/THT"
-			(at 0 0 0)
+			(at 0 0 90)
 			(layer "F.SilkS")
 			(hide yes)
@@
 		)
 		(fp_text user "${REFERENCE}"
-			(at 1.27 -2.72 0)
+			(at 1.27 -2.72 90)
 			(layer "F.Fab")
 			(effects
@@
 		)
 		(pad "1" thru_hole circle
-			(at 0 0)
+			(at 0 0 270)
 			(size 1.6 1.6)
 			(drill 0.8)
@@
 		)
 		(pad "2" thru_hole circle
-			(at 2.54 0)
+			(at 2.54 0 270)
 			(size 1.6 1.6)
 			(drill 0.8)
@@
 	)
 	(gr_rect
-		(start 182 82.5)
-		(end 190 97)
+		(start 75.5 70)
+		(end 132.5 91)
 		(stroke
 			(width 0.2)
@@
 		(layer "B.Cu")
 		(net "GND")
+	)
+	(segment
+		(start 106 82.67)
+		(end 104 80.67)
+		(width 0.2)
+		(layer "B.Cu")
+		(net "GND")
+	)
+	(segment
+		(start 104 80.67)
+		(end 104 80.5)
+		(width 0.2)
+		(layer "B.Cu")
+		(net "GND")
